Commit message: fix(pikachu)

File: resources/robots/Pikachu_V01/urdf/Pikachu_V01.urdf (robot description, URDF)
Before this commit: robot Pikachu_V01, 14 links, 13 joints
Links:
- added link imu, mass 0
- link Lankle_Link: geometry collision mesh filename=../meshes/Lankle_Link.STL; visual mesh filename=../meshes/Lankle_Link.STL
- link Larm_Link: geometry collision mesh filename=../meshes/Larm_Link.STL; visual mesh filename=../meshes/Larm_Link.STL
- link Lhip1_Link: geometry collision mesh filename=../meshes/Lhip1_Link.STL; visual mesh filename=../meshes/Lhip1_Link.STL
- link Lhip2_Link: geometry collision mesh filename=../meshes/Lhip2_Link.STL; visual mesh filename=../meshes/Lhip2_Link.STL
- link Lhip3_Link: geometry collision mesh filename=../meshes/Lhip3_Link.STL; visual mesh filename=../meshes/Lhip3_Link.STL
- link Lknee_Link: geometry collision mesh filename=../meshes/Lknee_Link.STL; visual mesh filename=../meshes/Lknee_Link.STL
- link Rankle_Link: geometry collision mesh filename=../meshes/Rankle_Link.STL; visual mesh filename=../meshes/Rankle_Link.STL
- link Rarm_Link: geometry collision mesh filename=../meshes/Rarm_Link.STL; visual mesh filename=../meshes/Rarm_Link.STL
- link Rhip1_Link: geometry collision mesh filename=../meshes/Rhip1_Link.STL; visual mesh filename=../meshes/Rhip1_Link.STL
- link Rhip2_Link: geometry collision mesh filename=../meshes/Rhip2_Link.STL; visual mesh filename=../meshes/Rhip2_Link.STL
- link Rhip3_Link: geometry collision mesh filename=../meshes/Rhip3_Link.STL; visual mesh filename=../meshes/Rhip3_Link.STL
- link Rknee_Link: geometry collision mesh filename=../meshes/Rknee_Link.STL; visual mesh filename=../meshes/Rknee_Link.STL
- link Tail_Link: geometry collision mesh filename=../meshes/Tail_Link.STL; visual mesh filename=../meshes/Tail_Link.STL
- link base_link: geometry collision mesh filename=../meshes/base_link.STL; visual mesh filename=../meshes/base_link.STL
Joints:
- removed joint Rarm_joint
- removed joint Rhip1_joint
- added joint Rarm_Joint: type continuous, parent base_link, child Rarm_Link, origin xyz=0.0200000000000008 -0.0809500000000023 0.205 rpy=1.57079632679488 1.5707963267949 0, axis 0 0 -1
- added joint Rhip1_Joint: type revolute, parent base_link, child Rhip1_Link, origin xyz=0 -0.0877000000000044 0 rpy=-1.5707963267949 0 -3.14159265358979, axis 0 0 -1, limit lower=-0.7 upper=2.7 effort=27 velocity=10
- added joint imu_joint: type fixed, parent base, child imu, origin xyz=-0.02557 0 0.04232 rpy=0 0 0, axis 0 0 0

Commit message: fix pikachu

File: resources/robots/Pikachu_V01/urdf/Pikachu_V01.urdf (robot description, URDF)
Before this commit: robot Pikachu_V01, 15 links, 14 joints
Links:
- removed link Lankle_Link
- removed link Larm_Link
- removed link Lhip1_Link
- removed link Lhip2_Link
- removed link Lhip3_Link
- removed link Lknee_Link
- removed link Rankle_Link
- removed link Rarm_Link
- removed link Rhip1_Link
- removed link Rhip2_Link
- removed link Rhip3_Link
- removed link Rknee_Link
- added link left_ankle_link, mass 0.0747132228410603; collision mesh filename=../meshes/left_ankle_link.STL; visual mesh filename=../meshes/left_ankle_link.STL
- added link left_arm_link, mass 0.132785524737081; collision mesh filename=../meshes/left_arm_link.STL; visual mesh filename=../meshes/left_arm_link.STL
- added link left_hip_pitch_link, mass 0.240283091885992; collision mesh filename=../meshes/left_hip_pitch_link.STL; visual mesh filename=../meshes/left_hip_pitch_link.STL
- added link left_hip_roll_link, mass 0.237453317125622; collision mesh filename=../meshes/left_hip_roll_link.STL; visual mesh filename=../meshes/left_hip_roll_link.STL
- added link left_hip_yaw_link, mass 0.329226275444801; collision mesh filename=../meshes/left_hip_yaw_link.STL; visual mesh filename=../meshes/left_hip_yaw_link.STL
- added link left_knee_link, mass 0.244244092244912; collision mesh filename=../meshes/left_knee_link.STL; visual mesh filename=../meshes/left_knee_link.STL
- added link right_ankle_link, mass 0.0747132228410604; collision mesh filename=../meshes/right_ankle_link.STL; visual mesh filename=../meshes/right_ankle_link.STL
- added link right_arm_link, mass 0.126051829781318; collision mesh filename=../meshes/right_arm_link.STL; visual mesh filename=../meshes/right_arm_link.STL
- added link right_hip_pitch_link, mass 0.240283091885992; collision mesh filename=../meshes/right_hip_pitch_link.STL; visual mesh filename=../meshes/right_hip_pitch_link.STL
- added link right_hip_roll_link, mass 0.237453317125623; collision mesh filename=../meshes/right_hip_roll_link.STL; visual mesh filename=../meshes/right_hip_roll_link.STL
- added link right_hip_yaw_link, mass 0.327324989928112; collision mesh filename=../meshes/right_hip_yaw_link.STL; visual mesh filename=../meshes/right_hip_yaw_link.STL
- added link right_knee_link, mass 0.244872851574774; collision mesh filename=../meshes/right_knee_link.STL; visual mesh filename=../meshes/right_knee_link.STL
Joints:
- removed joint Lankle_Joint
- removed joint Larm_Joint
- removed joint Lhip1_Joint
- removed joint Lhip2_Joint
- removed joint Lhip3_Joint
- removed joint Lknee_Joint
- removed joint Rankle_Joint
- removed joint Rarm_Joint
- removed joint Rhip1_Joint
- removed joint Rhip2_Joint
- removed joint Rhip3_Joint
- removed joint Rknee_Joint
- added joint left_ankle_joint: type revolute, parent left_knee_link, child left_ankle_link, origin xyz=0 0.1 0.00775000000000223 rpy=0 0 3.14159265358979, axis 0 0 -1, limit lower=-1.64 upper=1.64 effort=12.5 velocity=5
- added joint left_arm_joint: type continuous, parent base_link, child left_arm_link, origin xyz=0.0199999999999998 0.0809500000000004 0.205 rpy=-1.57079632679491 1.5707963267949 0, axis 0 0 -1
- added joint left_hip_pitch_joint: type revolute, parent base_link, child left_hip_pitch_link, origin xyz=0 0.0876999999999957 0 rpy=1.5707963267949 0 -3.14159265358979, axis 0 0 1, limit lower=-0.7 upper=2.7 effort=27 velocity=10
- added joint left_hip_roll_joint: type revolute, parent left_hip_pitch_link, child left_hip_roll_link, origin xyz=-0.0329999999998985 0 -0.0319999999999964 rpy=0 -1.5707963267949 0, axis 0 0 1, limit lower=-0.122 upper=0.139 effort=12.5 velocity=5
- added joint left_hip_yaw_joint: type revolute, parent left_hip_roll_link, child left_hip_yaw_link, origin xyz=0 -0.110499999999992 -0.0329999999999931 rpy=1.5707963267949 -1.5707963267949 0, axis 0 0 -1, limit lower=-0.261 upper=0.261 effort=12.5 velocity=5
- added joint left_knee_joint: type revolute, parent left_hip_yaw_link, child left_knee_link, origin xyz=0 -0.0402500000000001 0.038000000000008 rpy=1.5707963267949 0 0, axis 0 0 1, limit lower=0.04 upper=2.44 effort=12.5 velocity=5
- added joint right_ankle_joint: type revolute, parent right_knee_link, child right_ankle_link, origin xyz=0 -0.100000000000003 0.00775000000000253 rpy=3.14159265358979 0 3.14159265358979, axis 0 0 1, limit lower=-1.64 upper=1.64 effort=12.5 velocity=5
- added joint right_arm_joint: type continuous, parent base_link, child right_arm_link, origin xyz=0.0200000000000008 -0.0809500000000023 0.205 rpy=1.57079632679488 1.5707963267949 0, axis 0 0 -1
- added joint right_hip_pitch_joint: type revolute, parent base_link, child right_hip_pitch_link, origin xyz=0 -0.0877000000000044 0 rpy=-1.5707963267949 0 -3.14159265358979, axis 0 0 -1, limit lower=-0.7 upper=2.7 effort=27 velocity=10
- added joint right_hip_roll_joint: type revolute, parent right_hip_pitch_link, child right_hip_roll_link, origin xyz=-0.0330000000000126 0 -0.0320000000000056 rpy=3.14159265358979 1.5707963267949 0, axis 0 0 -1, limit lower=-0.122 upper=0.139 effort=12.5 velocity=5
- added joint right_hip_yaw_joint: type revolute, parent right_hip_roll_link, child right_hip_yaw_link, origin xyz=0 -0.110500000000004 -0.0330000000000059 rpy=1.5707963267949 -1.5707963267949 0, axis 0 0 -1, limit lower=-0.261 upper=0.261 effort=12.5 velocity=5
- added joint right_knee_joint: type revolute, parent right_hip_yaw_link, child right_knee_link, origin xyz=0 0.0419999999999997 0.037999999999996 rpy=-1.5707963267949 0 0, axis 0 0 -1, limit lower=0.04 upper=2.44 effort=12.5 velocity=5
